Commit message: Ch3-4 Second link Recap and Add Links Together

File: ros2_ws/src/my_robot_description/urdf/arm.urdf (robot description, URDF)
Before this commit: robot my_robot, 1 links, 0 joints
Links:
- added link shoulder_link; visual cylinder length=0.5 radius=0.1
Joints:
- added joint joint1: type revolute, parent base_link, child shoulder_link, origin xyz=0 0 0.1 rpy=0 0 0, axis 0 0 1, limit lower=-3.14 upper=3.14 effort=1000.0 velocity=1.0
