Commit message: Ch5-3 Connect the Gripper to the Arm

File: ros2_ws/src/my_robot_description/urdf/common_properties.xacro (robot description, xacro)
@@ -7,3 +7,9 @@
         <color rgba="0 0 0.5 1.0"/>
     </material>
+    <material name="dark_green">
+        <color rgba="0 0.4 0 1.0"/>
+    </material>
+    <material name="light_green">
+        <color rgba="0 0.6 0 1.0"/>
+    </material>
 </robot>

File: ros2_ws/src/my_robot_description/urdf/gripper.xacro (robot description, xacro)
@@ -1,10 +1,4 @@
 <?xml version="1.0"?>
-<robot name="temp" xmlns:xacro="http://www.ros.org/wiki/xacro">
-    <material name="dark_green">
-        <color rgba="0 0.4 0 1.0"/>
-    </material>
-    <material name="light_green">
-        <color rgba="0 0.6 0 1.0"/>
-    </material>
+<robot xmlns:xacro="http://www.ros.org/wiki/xacro">
     <link name="gripper_base_link">
         <visual>

File: ros2_ws/src/my_robot_description/urdf/my_robot.urdf.xacro (robot description, xacro)
@@ -3,3 +3,9 @@
     <xacro:include filename="common_properties.xacro" />
     <xacro:include filename="arm.xacro" />
+    <xacro:include filename="gripper.xacro" />
+    <joint name="gripper_base_joint" type="fixed">
+        <parent link="tool_link"/>
+        <child link="gripper_base_link"/>
+        <origin xyz="0 0 0" rpy="0 0 0"/>
+    </joint>
 </robot>
